Commit message: fixed exported urdf of realman_inspire_R include mimic, revolute joint and geometry file

File: Robots/Realman_Inspire/exported_urdf/Realman_Inspire_R/Realman_Inspire_R.urdf (robot description, URDF)
Before this commit: robot Realman_Inspire_R, 23 links, 22 joints
Links:
- link R_flange_link: geometry collision mesh filename=meshes/R_hand_flange.STL scale=1. 1. 1.; visual mesh filename=meshes/R_hand_flange.STL scale=1. 1. 1.
Joints:
- joint R_index_intermediate_joint: mimic (none) -> joint=R_index_proximal_joint multiplier=1 offset=0
- joint R_middle_intermediate_joint: mimic (none) -> joint=R_middle_proximal_joint multiplier=1 offset=0
- joint R_pinky_intermediate_joint: mimic (none) -> joint=R_pinky_proximal_joint multiplier=1 offset=0
- joint R_ring_intermediate_joint: mimic (none) -> joint=R_ring_proximal_joint multiplier=1 offset=0
- joint R_thumb_distal_joint: limit (none) -> lower=0 upper=1.2 effort=1 velocity=0.5; mimic (none) -> joint=R_thumb_proximal_pitch_joint multiplier=2.4 offset=0; type continuous -> revolute
- joint R_thumb_intermediate_joint: limit (none) -> lower=0 upper=0.8 effort=1 velocity=0.5; mimic (none) -> joint=R_thumb_proximal_pitch_joint multiplier=1.6 offset=0; type continuous -> revolute
