Commit message: finetune urdf of position of thumb bit a little bit

File: Robots/Realman_Inspire/urdf/Realman_Inspire_R/Realman_Inspire_R.urdf (robot description, URDF)
Before this commit: robot Realman_Inspire_R_mimic, 28 links, 27 joints
Joints:
- joint R_thumb_tip_joint: origin xyz=-0.006 0.020 -0.010 rpy=0 0 0 -> xyz=-0.006 0.013 -0.017 rpy=0 0 0
