Commit message: 20250103 usd and urdf update to fix the thumb collision issue

File: Robots/XHand/xhand_left.urdf (robot description, URDF)
Before this commit: robot xhand_left, 19 links, 18 joints
Links:
- added link base_link
- link left_hand_ee_link: geometry collision mesh filename=./meshes/left_hand_ee_link.STL; visual mesh filename=./meshes/left_hand_ee_link.STL
- link left_hand_index_bend_link: mass 0.0677836037392838 -> 0.0678358392130179; geometry visual mesh filename=./meshes/left_hand_index_bend_link.STL
- link left_hand_index_rota_link1: mass 0.0630216014538817 -> 0.0630023008144735; geometry collision mesh filename=./meshes/left_hand_index_rota_link1.STL; visual mesh filename=./meshes/left_hand_index_rota_link1.STL
- link left_hand_index_rota_link2: mass 0.0179923076570599 -> 0.017978306795458; geometry collision mesh filename=./meshes/left_hand_index_rota_link2.STL; visual mesh filename=./meshes/left_hand_index_rota_link2.STL
- link left_hand_index_rota_tip: geometry collision mesh filename=./meshes/left_hand_index_rota_tip.STL; visual mesh filename=./meshes/left_hand_index_rota_tip.STL
- link left_hand_link: mass 0.529961023577223 -> 0.529944310592205; geometry collision mesh filename=./meshes/left_hand_link.STL; visual mesh filename=./meshes/left_hand_link.STL
- link left_hand_mid_link1: mass 0.0630216000876532 -> 0.0630023022013301; geometry collision mesh filename=./meshes/left_hand_mid_link1.STL; visual mesh filename=./meshes/left_hand_mid_link1.STL
- link left_hand_mid_link2: mass 0.0179922971238626 -> 0.0179783068080897; geometry collision mesh filename=./meshes/left_hand_mid_link2.STL; visual mesh filename=./meshes/left_hand_mid_link2.STL
- link left_hand_mid_tip: geometry collision mesh filename=./meshes/left_hand_mid_tip.STL; visual mesh filename=./meshes/left_hand_mid_tip.STL
- link left_hand_pinky_link1: mass 0.0630216018833023 -> 0.0630022982822898; geometry collision mesh filename=./meshes/left_hand_pinky_link1.STL; visual mesh filename=./meshes/left_hand_pinky_link1.STL
- link left_hand_pinky_link2: mass 0.0179922893932107 -> 0.0179783067958151; geometry collision mesh filename=./meshes/left_hand_pinky_link2.STL; visual mesh filename=./meshes/left_hand_pinky_link2.STL
- link left_hand_pinky_tip: geometry collision mesh filename=./meshes/left_hand_pinky_tip.STL; visual mesh filename=./meshes/left_hand_pinky_tip.STL
- link left_hand_ring_link1: mass 0.0630216034004235 -> 0.0630023002480442; geometry collision mesh filename=./meshes/left_hand_ring_link1.STL; visual mesh filename=./meshes/left_hand_ring_link1.STL
- link left_hand_ring_link2: mass 0.0179923074393582 -> 0.0179783067963059; geometry collision mesh filename=./meshes/left_hand_ring_link2.STL; visual mesh filename=./meshes/left_hand_ring_link2.STL
- link left_hand_ring_tip: geometry collision mesh filename=./meshes/left_hand_ring_tip.STL; visual mesh filename=./meshes/left_hand_ring_tip.STL
- link left_hand_thumb_bend_link: mass 0.0098553409170395 -> 0.00988789386004912; geometry visual mesh filename=./meshes/left_hand_thumb_bend_link.STL
- link left_hand_thumb_rota_link1: mass 0.153197010050709 -> 0.153155034156758; geometry collision mesh filename=./meshes/left_hand_thumb_rota_link1.STL; visual mesh filename=./meshes/left_hand_thumb_rota_link1.STL
- link left_hand_thumb_rota_link2: mass 0.0374009578136616 -> 0.0374005336514977; geometry collision mesh filename=./meshes/left_hand_thumb_rota_link2.STL; visual mesh filename=./meshes/left_hand_thumb_rota_link2.STL
- link left_hand_thumb_rota_tip: geometry collision mesh filename=./meshes/left_hand_thumb_rota_tip.STL; visual mesh filename=./meshes/left_hand_thumb_rota_tip.STL
Joints:
- added joint base_link_joint: type fixed, parent base_link, child left_hand_link, origin xyz=0 0 0.0 rpy=0 0 0, axis 0 0 0
- joint left_hand_index_bend_joint: axis 0 1 0 -> 0 -1 0
- joint left_hand_index_rota_joint3: origin xyz=0 0 -0.0424999999999991 rpy=0 0 0 -> xyz=0 0 -0.0424999999999999 rpy=0 0 0
- joint left_hand_mid_joint3: origin xyz=0 0 -0.0424999999999995 rpy=0 0 0 -> xyz=0 0 -0.042500000000001 rpy=0 0 0
- joint left_hand_pinky_joint3: origin xyz=0 0 -0.0424999999999995 rpy=0 0 0 -> xyz=0 0 -0.0425 rpy=0 0 0
- joint left_hand_ring_joint3: origin xyz=0 0 -0.0425 rpy=0 0 0 -> xyz=0 0 -0.0424999999999995 rpy=0 0 0
- joint left_hand_thumb_rota_joint1: origin xyz=0.028599 -0.0083177 0.00178 rpy=-0.2618 0 -0.0407 -> xyz=0.0285986272129401 -0.00831765565268352 0.00177996188345445 rpy=-0.261799387798933 0 -0.0407002356493396
- joint left_hand_thumb_rota_joint2: origin xyz=0.0553 0 0 rpy=0 0 0 -> xyz=0.0552999999999999 0 0 rpy=0 0 0
- joint left_hand_thumb_rota_joint3: origin xyz=0.0504017317642718 0 0 rpy=0 0 0 -> xyz=0.0504024555173588 0 0 rpy=0 0 0

File: Robots/XHand/xhand_right.urdf (robot description, URDF)
Before this commit: robot xhand_right, 19 links, 18 joints
Links:
- added link base_link
- link right_hand_ee_link: geometry collision mesh filename=./meshes/right_hand_ee_link.STL; visual mesh filename=./meshes/right_hand_ee_link.STL
- link right_hand_index_bend_link: mass 0.0677836037392839 -> 0.0678358392130179; geometry visual mesh filename=./meshes/right_hand_index_bend_link.STL
- link right_hand_index_rota_link1: mass 0.0630216027459696 -> 0.0630022977710548; geometry collision mesh filename=./meshes/right_hand_index_rota_link1.STL; visual mesh filename=./meshes/right_hand_index_rota_link1.STL
- link right_hand_index_rota_link2: mass 0.0179923076356481 -> 0.0179783067962212; geometry collision mesh filename=./meshes/right_hand_index_rota_link2.STL; visual mesh filename=./meshes/right_hand_index_rota_link2.STL
- link right_hand_index_rota_tip: geometry collision mesh filename=./meshes/right_hand_index_rota_tip.STL; visual mesh filename=./meshes/right_hand_index_rota_tip.STL
- link right_hand_link: mass 0.530025137189824 -> 0.529993400990084; geometry collision mesh filename=./meshes/right_hand_link.STL; visual mesh filename=./meshes/right_hand_link.STL
- link right_hand_mid_link1: mass 0.0630216005457211 -> 0.0630022982853768; geometry collision mesh filename=./meshes/right_hand_mid_link1.STL; visual mesh filename=./meshes/right_hand_mid_link1.STL
- link right_hand_mid_link2: mass 0.0179923076388667 -> 0.0179783067957322; geometry collision mesh filename=./meshes/right_hand_mid_link2.STL; visual mesh filename=./meshes/right_hand_mid_link2.STL
- link right_hand_mid_tip: geometry collision mesh filename=./meshes/right_hand_mid_tip.STL; visual mesh filename=./meshes/right_hand_mid_tip.STL
- link right_hand_pinky_link1: mass 0.0630215991316208 -> 0.0630023023053313; geometry collision mesh filename=./meshes/right_hand_pinky_link1.STL; visual mesh filename=./meshes/right_hand_pinky_link1.STL
- link right_hand_pinky_link2: mass 0.0179923076462156 -> 0.017978306641324; geometry collision mesh filename=./meshes/right_hand_pinky_link2.STL; visual mesh filename=./meshes/right_hand_pinky_link2.STL
- link right_hand_pinky_tip: geometry collision mesh filename=./meshes/right_hand_pinky_tip.STL; visual mesh filename=./meshes/right_hand_pinky_tip.STL
- link right_hand_ring_link1: mass 0.0630216021699602 -> 0.0630023036931237; geometry collision mesh filename=./meshes/right_hand_ring_link1.STL; visual mesh filename=./meshes/right_hand_ring_link1.STL
- link right_hand_ring_link2: mass 0.0179922978524175 -> 0.0179783089787658; geometry collision mesh filename=./meshes/right_hand_ring_link2.STL; visual mesh filename=./meshes/right_hand_ring_link2.STL
- link right_hand_ring_tip: geometry collision mesh filename=./meshes/right_hand_ring_tip.STL; visual mesh filename=./meshes/right_hand_ring_tip.STL
- link right_hand_thumb_bend_link: mass 0.0098552942780609 -> 0.0098848519917835; geometry visual mesh filename=./meshes/right_hand_thumb_bend_link.STL
- link right_hand_thumb_rota_link1: mass 0.153264803291678 -> 0.153227150322195; geometry collision mesh filename=./meshes/right_hand_thumb_rota_link1.STL; visual mesh filename=./meshes/right_hand_thumb_rota_link1.STL
- link right_hand_thumb_rota_link2: mass 0.0374003730407777 -> 0.0374008322024407; geometry collision mesh filename=./meshes/right_hand_thumb_rota_link2.STL; visual mesh filename=./meshes/right_hand_thumb_rota_link2.STL
- link right_hand_thumb_rota_tip: geometry collision mesh filename=./meshes/right_hand_thumb_rota_tip.STL; visual mesh filename=./meshes/right_hand_thumb_rota_tip.STL
Joints:
- added joint base_link_joint: type fixed, parent base_link, child right_hand_link, origin xyz=0 0 0.0 rpy=0 0 0, axis 0 0 0
- joint right_hand_index_bend_joint: axis 0 1 0 -> 0 -1 0
- joint right_hand_index_rota_joint3: origin xyz=0 0 -0.0424999999999993 rpy=0 0 0 -> xyz=0 0 -0.0425000000000002 rpy=0 0 0
- joint right_hand_mid_joint3: origin xyz=0 0 -0.042107 rpy=0 0 0 -> xyz=0 0 -0.0424999999999994 rpy=0 0 0
- joint right_hand_pinky_joint3: origin xyz=0 0 -0.0425 rpy=0 0 0 -> xyz=0 0 -0.0424999999999994 rpy=0 0 0
- joint right_hand_thumb_rota_joint3: origin xyz=0.0504024546888781 0 0 rpy=0 0 0 -> xyz=0.0504024546888782 0 0 rpy=0 0 0
